Commit message: add the meshes

File: urdf/common_colors.xacro (robot description, xacro)
@@ -5,4 +5,4 @@
   <xacro:property name="color_fenrir_orange"   value="${ 234/255} ${ 91/255} ${ 20/255} 1.0" />
   <!-- Black -->
-  <xacro:property name="color_fenrir_black"   value="${ 10/255} ${ 10/255} ${ 10/255} 1.0" />
+  <xacro:property name="color_fenrir_black"   value="${ 30/255} ${ 30/255} ${ 30/255} 1.0" />
 </robot>

File: urdf/fenrir_macro.xacro (robot description, xacro)
@@ -7,5 +7,5 @@
         <origin xyz="0 0 0" rpy="0 0 0"/>
         <geometry>
-          <mesh filename="package://fenrir/meshes/visual/base_link.stl"/>
+          <mesh filename="package://fenrir/meshes/visual/base_link.stl" scale="0.01 0.01 0.01"/>
         </geometry>
         <xacro:material_fenrir_black/>
@@ -14,5 +14,5 @@
         <origin xyz="0 0 0" rpy="0 0 0"/>
         <geometry>
-          <mesh filename="package://fenrir/meshes/collision/base_link.stl"/>
+          <mesh filename="package://fenrir/meshes/collision/base_link.stl" scale="0.01 0.01 0.01"/>
         </geometry>
       </collision>
@@ -22,5 +22,5 @@
         <origin xyz="0 0 0" rpy="0 0 0"/>
         <geometry>
-          <mesh filename="package://fenrir/meshes/visual/disk.stl"/>
+          <mesh filename="package://fenrir/meshes/visual/disk.stl" scale="0.01 0.01 0.01"/>
         </geometry>
         <xacro:material_fenrir_black />
@@ -29,5 +29,5 @@
         <origin xyz="0 0 0" rpy="0 0 0"/>
         <geometry>
-          <mesh filename="package://fenrir/meshes/collision/disk.stl"/>
+          <mesh filename="package://fenrir/meshes/collision/disk.stl" scale="0.01 0.01 0.01"/>
         </geometry>
       </collision>
@@ -35,7 +35,7 @@
     <link name="${prefix}lower_arm">
       <visual>
-        <origin xyz="0 0 0" rpy="0 0 0"/>
+        <origin xyz="0 0.022 0" rpy="0 0 0"/>
         <geometry>
-          <mesh filename="package://fenrir/meshes/visual/lower_arm.stl"/>
+          <mesh filename="package://fenrir/meshes/visual/lower_arm.stl" scale="0.01 0.01 0.01"/>
         </geometry>
         <xacro:material_fenrir_black />
@@ -44,5 +44,5 @@
         <origin xyz="0 0 0" rpy="0 0 0"/>
         <geometry>
-          <mesh filename="package://fenrir/meshes/collision/lower_arm.stl"/>
+          <mesh filename="package://fenrir/meshes/collision/lower_arm.stl" scale="0.01 0.01 0.01"/>
         </geometry>
       </collision>
@@ -52,5 +52,5 @@
         <origin xyz="0 0 0" rpy="0 0 0"/>
         <geometry>
-          <mesh filename="package://fenrir/meshes/visual/forearm.stl"/>
+          <mesh filename="package://fenrir/meshes/visual/forearm.stl" scale="0.01 0.01 0.01"/>
         </geometry>
         <xacro:material_fenrir_orange />
@@ -59,5 +59,5 @@
         <origin xyz="0 0 0" rpy="0 0 0"/>
         <geometry>
-          <mesh filename="package://fenrir/meshes/collision/forearm.stl"/>
+          <mesh filename="package://fenrir/meshes/collision/forearm.stl" scale="0.01 0.01 0.01"/>
         </geometry>
       </collision>
@@ -67,5 +67,5 @@
         <origin xyz="0 0 0" rpy="0 0 0"/>
         <geometry>
-          <mesh filename="package://fenrir/meshes/visual/end_effector.stl"/>
+          <mesh filename="package://fenrir/meshes/visual/end_effector.stl" scale="0.01 0.01 0.01"/>
         </geometry>
         <xacro:material_fenrir_black />
@@ -74,5 +74,5 @@
         <origin xyz="0 0 0" rpy="0 0 0"/>
         <geometry>
-          <mesh filename="package://fenrir/meshes/collision/end_effector.stl"/>
+          <mesh filename="package://fenrir/meshes/collision/end_effector.stl" scale="0.01 0.01 0.01"/>
         </geometry>
       </collision>
@@ -80,5 +80,5 @@
     <!-- joints: main serial chain -->
     <joint name="${prefix}base" type="revolute">
-      <origin xyz="0 0 0.200" rpy="0 0 0"/>
+      <origin xyz="0 0 0.080" rpy="0 0 0"/>
       <parent link="${prefix}base_link"/>
       <child link="${prefix}disk"/>
@@ -87,5 +87,5 @@
     </joint>
     <joint name="${prefix}sholder" type="revolute">
-      <origin xyz="0 0 0.600" rpy="0 0 0"/>
+      <origin xyz="0 0 0.080" rpy="0 0 0"/>
       <parent link="${prefix}disk"/>
       <child link="${prefix}lower_arm"/>
@@ -94,5 +94,5 @@
     </joint>
     <joint name="${prefix}elbow" type="revolute">
-      <origin xyz="0 0 0.450" rpy="0 0 0"/>
+      <origin xyz="0 0.001 0.195" rpy="0 0 0"/>
       <parent link="${prefix}lower_arm"/>
       <child link="${prefix}forearm"/>
@@ -101,5 +101,5 @@
     </joint>
     <joint name="${prefix}wrist" type="revolute">
-      <origin xyz="0 0 0.200" rpy="0 0 0"/>
+      <origin xyz="0 0 0.15" rpy="0 0 0"/>
       <parent link="${prefix}forearm"/>
       <child link="${prefix}end_effector"/>
