Commit message: rename some files

File: urdf/fenrir.urdf (robot description, URDF)
Before this commit: robot Fenrir, 5 links, 4 joints
Links:
- link base_link: geometry collision mesh filename=package://fenrir/meshes/collision/base_link.stl scale=0.01 0.01 0.01; visual mesh filename=package://fenrir/meshes/visual/base_link.stl scale=0.01 0.01 0.01
- link disk: geometry collision mesh filename=package://fenrir/meshes/collision/disk.stl scale=0.01 0.01 0.01; visual mesh filename=package://fenrir/meshes/visual/disk.stl scale=0.01 0.01 0.01
- link end_effector: geometry collision mesh filename=package://fenrir/meshes/collision/end_effector.stl scale=0.01 0.01 0.01; visual mesh filename=package://fenrir/meshes/visual/end_effector.stl scale=0.01 0.01 0.01
- link forearm: geometry collision mesh filename=package://fenrir/meshes/collision/forearm.stl scale=0.01 0.01 0.01; visual mesh filename=package://fenrir/meshes/visual/forearm.stl scale=0.01 0.01 0.01
- link lower_arm: geometry collision mesh filename=package://fenrir/meshes/collision/lower_arm.stl scale=0.01 0.01 0.01; visual mesh filename=package://fenrir/meshes/visual/lower_arm.stl scale=0.01 0.01 0.01
Joints:
- joint base: origin xyz=0 0 0.200 rpy=0 0 0 -> xyz=0 0 0.080 rpy=0 0 0
- joint elbow: origin xyz=0 0 0.450 rpy=0 0 0 -> xyz=0 0.001 0.195 rpy=0 0 0
- joint sholder: origin xyz=0 0 0.600 rpy=0 0 0 -> xyz=0 0 0.080 rpy=0 0 0
- joint wrist: origin xyz=0 0 0.200 rpy=0 0 0 -> xyz=0 0 0.15 rpy=0 0 0

Commit message: add simulation driver

File: urdf/fenrir.urdf (robot description, URDF)
Before this commit: robot Fenrir, 5 links, 4 joints
Joints:
- removed joint base
- removed joint elbow
- removed joint sholder
- removed joint wrist
- added joint Base: type revolute, parent base_link, child disk, origin xyz=0 0 0.080 rpy=0 0 0, axis 0 0 1, limit lower=-2.967 upper=2.967 effort=0 velocity=4.01
- added joint Elbow: type revolute, parent lower_arm, child forearm, origin xyz=0 0.001 0.195 rpy=0 0 0, axis 0 -1 0, limit lower=-3.14 upper=4.66 effort=0 velocity=4.01
- added joint Shoulder: type revolute, parent disk, child lower_arm, origin xyz=0 0 0.080 rpy=0 0 0, axis 0 1 0, limit lower=-1.57 upper=2.79 effort=0 velocity=3.93
- added joint Wrist: type revolute, parent forearm, child end_effector, origin xyz=0 0 0.15 rpy=0 0 0, axis -1 0 0, limit lower=-3.31 upper=3.31 effort=0 velocity=7.50

Commit message: Fix 0 position URDF

File: urdf/fenrir.urdf (robot description, URDF)
Before this commit: robot Fenrir, 5 links, 4 joints
Joints:
- joint Elbow: limit lower=-3.14 upper=4.66 effort=0 velocity=4.01 -> lower=-6.14 upper=6.66 effort=0 velocity=4.01
- joint Shoulder: limit lower=-1.57 upper=2.79 effort=0 velocity=3.93 -> lower=-3.57 upper=3.79 effort=0 velocity=3.93

File: urdf/fenrir_macro.xacro (robot description, xacro)
@@ -210,16 +210,16 @@
     </joint>
     <joint name="${prefix}Shoulder" type="revolute">
-      <origin xyz="0 0 0.080" rpy="0 0 0"/>
+      <origin xyz="0 0 0.080" rpy="0 3.1415 0"/>
       <parent link="${prefix}disk"/>
       <child link="${prefix}lower_arm"/>
       <axis xyz="0 1 0"/>
-      <limit lower="-1.57" upper="2.79" effort="0" velocity="3.93"/>
+      <limit lower="-3.57" upper="3.79" effort="0" velocity="3.93"/>
     </joint>
     <joint name="${prefix}Elbow" type="revolute">
-      <origin xyz="0 0.001 0.195" rpy="0 0 0"/>
+      <origin xyz="0 0.001 0.195" rpy="0 3.1415 0"/>
       <parent link="${prefix}lower_arm"/>
       <child link="${prefix}forearm"/>
       <axis xyz="0 -1 0"/>
-      <limit lower="-3.14" upper="4.66" effort="0" velocity="4.01"/>
+      <limit lower="-6.14" upper="6.66" effort="0" velocity="4.01"/>
     </joint>
     <joint name="${prefix}Wrist" type="revolute">

Commit message: bla

File: urdf/fenrir.urdf (robot description, URDF)
Before this commit: robot Fenrir, 5 links, 4 joints
Links:
- removed link end_effector
- added link driving_gear; collision mesh filename=package://fenrir/meshes/collision/driving_gear.stl scale=0.01 0.01 0.01; visual mesh filename=package://fenrir/meshes/visual/driving_gear.stl scale=0.01 0.01 0.01
- added link gripper_base; collision mesh filename=package://fenrir/meshes/collision/ManipulatorServoHolder.stl scale=0.01 0.01 0.01; visual mesh filename=package://fenrir/meshes/visual/ManipulatorServoHolder.stl scale=0.01 0.01 0.01
- added link gripper_tip; collision mesh filename=package://fenrir/meshes/collision/gripperTip.stl scale=0.01 0.01 0.01; visual mesh filename=package://fenrir/meshes/visual/gripperTip.stl scale=0.01 0.01 0.01
- added link rod; collision mesh filename=package://fenrir/meshes/collision/secondaryRod.stl scale=0.01 0.01 0.01; visual mesh filename=package://fenrir/meshes/visual/secondaryRod.stl scale=0.01 0.01 0.01
- added link rod_slave; collision mesh filename=package://fenrir/meshes/collision/secondaryRod.stl scale=0.01 0.01 0.01; visual mesh filename=package://fenrir/meshes/visual/secondaryRod.stl scale=0.01 0.01 0.01
- added link slave_gear; collision mesh filename=package://fenrir/meshes/collision/slave_gear.stl scale=0.01 0.01 0.01; visual mesh filename=package://fenrir/meshes/visual/slave_gear.stl scale=0.01 0.01 0.01
- added link tip_slave; collision mesh filename=package://fenrir/meshes/collision/gripperTip.stl scale=0.01 0.01 0.01; visual mesh filename=package://fenrir/meshes/visual/gripperTip.stl scale=0.01 0.01 0.01
- link forearm: geometry collision mesh filename=package://fenrir/meshes/collision/forearm.stl scale=0.01 0.01 0.01; visual mesh filename=package://fenrir/meshes/visual/ax-12.stl scale=0.01 0.01 0.01
Joints:
- added joint Gripper: type revolute, parent gripper_base, child driving_gear, origin xyz=0 0.014 0.0262 rpy=0.40 0 0, axis -1 0 0, limit lower=-3.31 upper=3.31 effort=0 velocity=7.50
- added joint Gripper_slave: type revolute, parent gripper_base, child slave_gear, origin xyz=0 -0.0135 0.0262 rpy=-0.40 0 0, axis -1 0 0, limit lower=-3.31 upper=3.31 effort=0 velocity=7.50, mimic joint=Gripper multiplier=-1 offset=0
- added joint Rod_left: type revolute, parent gripper_base, child rod, origin xyz=0 0.0124 0.054 rpy=0.40 0 0, axis -1 0 0, limit lower=-3.31 upper=3.31 effort=0 velocity=7.50, mimic joint=Gripper multiplier=1.26 offset=0
- added joint Rod_right: type revolute, parent gripper_base, child rod_slave, origin xyz=0 -0.0115 0.054 rpy=-0.40 0 0, axis -1 0 0, limit lower=-3.31 upper=3.31 effort=0 velocity=7.50, mimic joint=Gripper multiplier=-1.26 offset=0
- added joint Tip_left: type revolute, parent driving_gear, child gripper_tip, origin xyz=0 0.052 0 rpy=-0.07 0 0, axis -1 0 0, limit lower=-3.31 upper=3.31 effort=0 velocity=7.50, mimic joint=Gripper multiplier=-0.8 offset=0
- added joint Tip_right: type revolute, parent slave_gear, child tip_slave, origin xyz=0 -0.052 0 rpy=0.07 0 0, axis -1 0 0, limit lower=-3.31 upper=3.31 effort=0 velocity=7.50, mimic joint=Gripper multiplier=0.8 offset=0
- joint Elbow: origin xyz=0 0.001 0.195 rpy=0 0 0 -> xyz=0 0.001 0.195 rpy=0 2.4 0
- joint Shoulder: origin xyz=0 0 0.080 rpy=0 0 0 -> xyz=0 -0.001 0.089 rpy=0 -0.6 0
- joint Wrist: axis -1 0 0 -> 0 0 -1; child end_effector -> gripper_base; origin xyz=0 0 0.15 rpy=0 0 0 -> xyz=0 0 0.19 rpy=0 0 0

File: urdf/fenrir_macro.xacro (robot description, xacro)
@@ -210,5 +210,5 @@
     </joint>
     <joint name="${prefix}Shoulder" type="revolute">
-      <origin xyz="0 0 0.080" rpy="0 0 0"/>
+      <origin xyz="0 -0.001 0.089" rpy="0 -0.6 0"/>
       <parent link="${prefix}disk"/>
       <child link="${prefix}lower_arm"/>
@@ -217,5 +217,5 @@
     </joint>
     <joint name="${prefix}Elbow" type="revolute">
-      <origin xyz="0 0.001 0.195" rpy="0 0 0"/>
+      <origin xyz="0 0.001 0.195" rpy="0 2.4 0"/>
       <parent link="${prefix}lower_arm"/>
       <child link="${prefix}forearm"/>
